Commit message: Added voice robot package and ROS2 navigation integration

File: src/my_bot/urdf/my_bot.urdf (robot description, URDF)
Before this commit: robot delivery_bot, 6 links, 5 joints
Links:
- link base_link: mass 5.0 -> 3.0
- link left_wheel: mass 1.0 -> 0.3; geometry collision cylinder length=0.08 radius=0.07; visual cylinder length=0.08 radius=0.07
- link right_wheel: mass 1.0 -> 0.3; geometry collision cylinder length=0.08 radius=0.07; visual cylinder length=0.08 radius=0.07
Joints:
- joint base_joint: origin xyz=0 0 0.05 rpy=0 0 0 -> xyz=0 0 0.06 rpy=0 0 0
- joint caster_joint: origin xyz=-0.15 0 -0.02 -> xyz=-0.15 0 -0.06
- joint left_wheel_joint: origin xyz=0 0.20 -0.02 rpy=0 0 0 -> xyz=0 0.20 -0.03 rpy=0 0 0
- joint right_wheel_joint: origin xyz=0 -0.20 -0.02 rpy=0 0 0 -> xyz=0 -0.20 -0.03 rpy=0 0 0
